Commit message: Rename variables and macros to Vietnamese

File: description/cauhinh_robot.xacro (robot description, xacro)
@@ -1,12 +1,12 @@
 <?xml version="1.0"?>
 <robot xmlns:xacro="http://www.ros.org/wiki/xacro" name="robot">
-    <xacro:include filename="inertial_macros.xacro"/>
+    <xacro:include filename="quan_tinh_macros.xacro"/>
     <xacro:property name="dai" value="0.25"/>
     <xacro:property name="rong" value="0.23"/>
     <xacro:property name="cao" value="0.15"/>
     <xacro:property name="KhoiLuongKhung" value="1.0"/>
-    <xacro:property name="DoRongBanhxe" value="0.027"/>
-    <xacro:property name="BanKinBanhxe" value="0.0325"/>
-    <xacro:property name="KL_Banhxe" value="0.1"/>
+    <xacro:property name="do_rong_banh_xe" value="0.027"/>
+    <xacro:property name="ban_kinh_banh_xe" value="0.0325"/>
+    <xacro:property name="khoi_luong_banh_xe" value="0.1"/>
     <xacro:property name="BK_BDH" value="0.015"/>
     <xacro:property name="KL_BDH" value="0.1"/>
@@ -43,7 +43,7 @@
             </geometry>
         </collision>
-            <xacro:inertial_box mass="${KhoiLuongKhung}" x="${dai}" y="${rong}" z="${cao}">
+            <xacro:quan_tinh_hinh_hop mass="${KhoiLuongKhung}" x="${dai}" y="${rong}" z="${cao}">
             <origin xyz="${dai/2} 0 ${cao/2}" rpy="0 0 0"/>
-        </xacro:inertial_box>
+        </xacro:quan_tinh_hinh_hop>
     </link>
     <gazebo reference="khung">
@@ -59,5 +59,5 @@
         <visual>
             <geometry>
-                <cylinder radius="${BanKinBanhxe}" length="${DoRongBanhxe}"/>
+                <cylinder radius="${ban_kinh_banh_xe}" length="${do_rong_banh_xe}"/>
             </geometry>
             <material name="blue"/>
@@ -65,10 +65,10 @@
         <collision>
             <geometry>
-                <cylinder radius="${BanKinBanhxe}" length="${DoRongBanhxe}"/>
+                <cylinder radius="${ban_kinh_banh_xe}" length="${do_rong_banh_xe}"/>
             </geometry>
         </collision>
-        <xacro:inertial_cylinder mass="${KL_Banhxe}" length="${DoRongBanhxe}" radius="${BanKinBanhxe}">
+        <xacro:quan_tinh_hinh_tru mass="${khoi_luong_banh_xe}" length="${do_rong_banh_xe}" radius="${ban_kinh_banh_xe}">
             <origin xyz="0 0 0" rpy="0 0 0"/>
-        </xacro:inertial_cylinder>
+        </xacro:quan_tinh_hinh_tru>
     </link>
     <gazebo reference="Banh_trai">
@@ -84,5 +84,5 @@
         <visual>
             <geometry>
-                <cylinder radius="${BanKinBanhxe}" length="${DoRongBanhxe}"/>
+                <cylinder radius="${ban_kinh_banh_xe}" length="${do_rong_banh_xe}"/>
             </geometry>
             <material name="blue"/>
@@ -90,10 +90,10 @@
         <collision>
             <geometry>
-                <cylinder radius="${BanKinBanhxe}" length="${DoRongBanhxe}"/>
+                <cylinder radius="${ban_kinh_banh_xe}" length="${do_rong_banh_xe}"/>
             </geometry>
         </collision>
-        <xacro:inertial_cylinder mass="${KL_Banhxe}" length="${DoRongBanhxe}" radius="${BanKinBanhxe}">
+        <xacro:quan_tinh_hinh_tru mass="${khoi_luong_banh_xe}" length="${do_rong_banh_xe}" radius="${ban_kinh_banh_xe}">
             <origin xyz="0 0 0" rpy="0 0 0"/>
-        </xacro:inertial_cylinder>
+        </xacro:quan_tinh_hinh_tru>
     </link>
     <gazebo reference="Banh_phai">
@@ -118,7 +118,7 @@
             <material name="black"/>
         </collision>
-        <xacro:inertial_sphere mass="${KL_BDH}" radius="${BK_BDH}">
+        <xacro:quan_tinh_hinh_cau mass="${KL_BDH}" radius="${BK_BDH}">
             <origin xyz="0 0 0" rpy="0 0 0"/>
-        </xacro:inertial_sphere>
+        </xacro:quan_tinh_hinh_cau>
     </link>
     <gazebo reference="BDH_trc">
@@ -145,7 +145,7 @@
             <material name="black"/>
         </collision>
-        <xacro:inertial_sphere mass="${KL_BDH}" radius="${BK_BDH}">
+        <xacro:quan_tinh_hinh_cau mass="${KL_BDH}" radius="${BK_BDH}">
             <origin xyz="0 0 0" rpy="0 0 0"/>
-        </xacro:inertial_sphere>
+        </xacro:quan_tinh_hinh_cau>
     </link>
     <gazebo reference="BDH_sau">

File: description/gazebo_control.xacro (robot description, xacro)
@@ -8,7 +8,7 @@
             <!-- KHoảng cách 2 bánh xe -->
             <wheel_separation>${rong}</wheel_separation>
-            <!-- Duong kinh banh xe -->
-            <wheel_diameter>${BanKinBanhxe * 2}</wheel_diameter>
-            <!-- Limits  Giới hạn gia tốc và momen xoắn-->
+            <!-- Đường kính bánh xe -->
+            <wheel_diameter>${ban_kinh_banh_xe * 2}</wheel_diameter>
+            <!-- Giới hạn gia tốc và momen xoắn -->
             <max_wheel_torque>200</max_wheel_torque>
             <max_wheel_acceleration>10.0</max_wheel_acceleration>

File: description/lidar.xacro (robot description, xacro)
@@ -18,7 +18,7 @@
             </geometry>
         </collision>
-        <xacro:inertial_cylinder mass="0.1" length="0.04" radius="0.05">
+        <xacro:quan_tinh_hinh_tru mass="0.1" length="0.04" radius="0.05">
             <origin xyz="0 0 0" rpy="0 0 0"/>
-        </xacro:inertial_cylinder>
+        </xacro:quan_tinh_hinh_tru>
     </link>
         <!-- NHO BAT TAT MO PHONG LIDAR true false-->

File: description/quan_tinh_macros.xacro (robot description, xacro)
@@ -1,7 +1,7 @@
 <?xml version="1.0"?>
 <robot xmlns:xacro="http://www.ros.org/wiki/xacro" >
-    <!-- Day la file quan tinh -->
-    <!-- Quan tinh hinh tru -->
-    <xacro:macro name="inertial_sphere" params="mass radius *origin">
+    <!-- Đây là file quản tính -->
+    <!-- Quán tính hình cầu -->
+    <xacro:macro name="quan_tinh_hinh_cau" params="mass radius *origin">
         <inertial>
             <xacro:insert_block name="origin"/>
@@ -12,6 +12,6 @@
         </inertial>
     </xacro:macro>
-    <!-- Quan tinh hinh hop -->
-    <xacro:macro name="inertial_box" params="mass x y z *origin">
+    <!-- Quán tính hình hộp -->
+    <xacro:macro name="quan_tinh_hinh_hop" params="mass x y z *origin">
         <inertial>
             <xacro:insert_block name="origin"/>
@@ -22,6 +22,6 @@
         </inertial>
     </xacro:macro>
-    <!-- Quan tinh hinh tru -->
-    <xacro:macro name="inertial_cylinder" params="mass length radius *origin">
+    <!-- Quán tính hình trụ -->
+    <xacro:macro name="quan_tinh_hinh_tru" params="mass length radius *origin">
         <inertial>
             <xacro:insert_block name="origin"/>

File: description/robot.urdf.xacro (robot description, xacro)
@@ -2,5 +2,5 @@
 <robot xmlns:xacro="http://www.ros.org/wiki/xacro"  name="robot">
     <xacro:arg name="Su_Dung_ros2_control" default="true"/>
-    <xacro:include filename="robot_core.xacro" />
+    <xacro:include filename="cauhinh_robot.xacro" />
     <xacro:include filename="gazebo_control.xacro" />
     <xacro:include filename="lidar.xacro" />
